Commit message: init

File: urdf/Cogni-robot.urdf (robot description, URDF)
Before this commit: robot Cogni-robot, 36 links, 35 joints
Links:
- link Prehenseur_fifty_fifty_Main_right_v1_1: geometry collision mesh filename=../../meshes/Prehenseur_fifty_fifty_Main_right_v1_1.stl scale=0.001 0.001 0.001; visual mesh filename=../../meshes/Prehenseur_fifty_fifty_Main_right_v1_1.stl scale=0.001 0.001 0.001
- link Prehenseur_fifty_fifty_Main_right_v1__1__1: geometry collision mesh filename=../../meshes/Prehenseur_fifty_fifty_Main_right_v1__1__1.stl scale=0.001 0.001 0.001; visual mesh filename=../../meshes/Prehenseur_fifty_fifty_Main_right_v1__1__1.stl scale=0.001 0.001 0.001
- link Prehenseur_fifty_fifty_Pousse_right_v1_1: geometry collision mesh filename=../../meshes/Prehenseur_fifty_fifty_Pousse_right_v1_1.stl scale=0.001 0.001 0.001; visual mesh filename=../../meshes/Prehenseur_fifty_fifty_Pousse_right_v1_1.stl scale=0.001 0.001 0.001
- link Prehenseur_fifty_fifty_Pousse_right_v1__1__1: geometry collision mesh filename=../../meshes/Prehenseur_fifty_fifty_Pousse_right_v1__1__1.s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 scale=0.001 0.001 0.001; visual mesh filename=../../meshes/Prehenseur_fifty_fifty_Pousse_right_v1__1__1.s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 scale=0.001 0.001 0.001
- link arm_connector_Feetech_v1_1: geometry collision mesh filename=../../meshes/arm_connector_Feetech_v1_1.stl scale=0.001 0.001 0.001; visual mesh filename=../../meshes/arm_connector_Feetech_v1_1.stl scale=0.001 0.001 0.001
- link arm_connector_Feetech_v1__1__1: geometry collision mesh filename=../../meshes/arm_connector_Feetech_v1__1__1.stl scale=0.001 0.001 0.001; visual mesh filename=../../meshes/arm_connector_Feetech_v1__1__1.stl scale=0.001 0.001 0.001
- link avant_bras_left_1: geometry collision mesh filename=../../meshes/avant_bras_left_1.stl scale=0.001 0.001 0.001; visual mesh filename=../../meshes/avant_bras_left_1.stl scale=0.001 0.001 0.001
- link avant_bras_right_v1_1: geometry collision mesh filename=../../meshes/avant_bras_right_v1_1.stl scale=0.001 0.001 0.001; visual mesh filename=../../meshes/avant_bras_right_v1_1.stl scale=0.001 0.001 0.001
- link base_link: geometry collision mesh filename=../../meshes/base_link.stl scale=0.001 0.001 0.001; visual mesh filename=../../meshes/base_link.stl scale=0.001 0.001 0.001
- link chest_1: geometry collision mesh filename=../../meshes/chest_1.stl scale=0.001 0.001 0.001; visual mesh filename=../../meshes/chest_1.stl scale=0.001 0.001 0.001
- link double_rotation_link_double_feetech_v1_1: geometry collision mesh filename=../../meshes/double_rotation_link_double_feetech_v1_1.stl scale=0.001 0.001 0.001; visual mesh filename=../../meshes/double_rotation_link_double_feetech_v1_1.stl scale=0.001 0.001 0.001
- link double_rotation_link_double_feetech_v1__1__1: geometry collision mesh filename=../../meshes/double_rotation_link_double_feetech_v1__1__1.s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 scale=0.001 0.001 0.001; visual mesh filename=../../meshes/double_rotation_link_double_feetech_v1__1__1.s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 scale=0.001 0.001 0.001
- link head_back_v2_1: geometry collision mesh filename=../../meshes/head_back_v2_1.stl scale=0.001 0.001 0.001; visual mesh filename=../../meshes/head_back_v2_1.stl scale=0.001 0.001 0.001
- link head_face_v1_1: geometry collision mesh filename=../../meshes/head_face_v1_1.stl scale=0.001 0.001 0.001; visual mesh filename=../../meshes/head_face_v1_1.stl scale=0.001 0.001 0.001
- link neck_v2_1: geometry collision mesh filename=../../meshes/neck_v2_1.stl scale=0.001 0.001 0.001; visual mesh filename=../../meshes/neck_v2_1.stl scale=0.001 0.001 0.001
- link screen_v1_1: geometry collision mesh filename=../../meshes/screen_v1_1.stl scale=0.001 0.001 0.001; visual mesh filename=../../meshes/screen_v1_1.stl scale=0.001 0.001 0.001
- link servo-sts3215-2_1: geometry collision mesh filename=../../meshes/servo-sts3215-2_1.stl scale=0.001 0.001 0.001; visual mesh filename=../../meshes/servo-sts3215-2_1.stl scale=0.001 0.001 0.001
- link servo_sts3215-2_1: geometry collision mesh filename=../../meshes/servo_sts3215-2_1.stl scale=0.001 0.001 0.001; visual mesh filename=../../meshes/servo_sts3215-2_1.stl scale=0.001 0.001 0.001
- link servo_sts3215_v1_1: geometry collision mesh filename=../../meshes/servo_sts3215_v1_1.stl scale=0.001 0.001 0.001; visual mesh filename=../../meshes/servo_sts3215_v1_1.stl scale=0.001 0.001 0.001
- link servo_sts3215_v1__10__1: geometry collision mesh filename=../../meshes/servo_sts3215_v1__10__1.stl scale=0.001 0.001 0.001; visual mesh filename=../../meshes/servo_sts3215_v1__10__1.stl scale=0.001 0.001 0.001
- link servo_sts3215_v1__11__1: geometry collision mesh filename=../../meshes/servo_sts3215_v1__11__1.stl scale=0.001 0.001 0.001; visual mesh filename=../../meshes/servo_sts3215_v1__11__1.stl scale=0.001 0.001 0.001
- link servo_sts3215_v1__12__1: geometry collision mesh filename=../../meshes/servo_sts3215_v1__12__1.stl scale=0.001 0.001 0.001; visual mesh filename=../../meshes/servo_sts3215_v1__12__1.stl scale=0.001 0.001 0.001
- link servo_sts3215_v1__1__1: geometry collision mesh filename=../../meshes/servo_sts3215_v1__1__1.stl scale=0.001 0.001 0.001; visual mesh filename=../../meshes/servo_sts3215_v1__1__1.stl scale=0.001 0.001 0.001
- link servo_sts3215_v1__2__1: geometry collision mesh filename=../../meshes/servo_sts3215_v1__2__1.stl scale=0.001 0.001 0.001; visual mesh filename=../../meshes/servo_sts3215_v1__2__1.stl scale=0.001 0.001 0.001
- link servo_sts3215_v1__3__1: geometry collision mesh filename=../../meshes/servo_sts3215_v1__3__1.stl scale=0.001 0.001 0.001; visual mesh filename=../../meshes/servo_sts3215_v1__3__1.stl scale=0.001 0.001 0.001
- link servo_sts3215_v1__4__1: geometry collision mesh filename=../../meshes/servo_sts3215_v1__4__1.stl scale=0.001 0.001 0.001; visual mesh filename=../../meshes/servo_sts3215_v1__4__1.stl scale=0.001 0.001 0.001
- link servo_sts3215_v1__5__1: geometry collision mesh filename=../../meshes/servo_sts3215_v1__5__1.stl scale=0.001 0.001 0.001; visual mesh filename=../../meshes/servo_sts3215_v1__5__1.stl scale=0.001 0.001 0.001
- link servo_sts3215_v1__6__1: geometry collision mesh filename=../../meshes/servo_sts3215_v1__6__1.stl scale=0.001 0.001 0.001; visual mesh filename=../../meshes/servo_sts3215_v1__6__1.stl scale=0.001 0.001 0.001
- link servo_sts3215_v1__7__1: geometry collision mesh filename=../../meshes/servo_sts3215_v1__7__1.stl scale=0.001 0.001 0.001; visual mesh filename=../../meshes/servo_sts3215_v1__7__1.stl scale=0.001 0.001 0.001
- link servo_sts3215_v1__8__1: geometry collision mesh filename=../../meshes/servo_sts3215_v1__8__1.stl scale=0.001 0.001 0.001; visual mesh filename=../../meshes/servo_sts3215_v1__8__1.stl scale=0.001 0.001 0.001
- link servo_sts3215_v1__9__1: geometry collision mesh filename=../../meshes/servo_sts3215_v1__9__1.stl scale=0.001 0.001 0.001; visual mesh filename=../../meshes/servo_sts3215_v1__9__1.stl scale=0.001 0.001 0.001
- link shoulder_left_v1_1: geometry collision mesh filename=../../meshes/shoulder_left_v1_1.stl scale=0.001 0.001 0.001; visual mesh filename=../../meshes/shoulder_left_v1_1.stl scale=0.001 0.001 0.001
- link shoulder_right_v1_1: geometry collision mesh filename=../../meshes/shoulder_right_v1_1.stl scale=0.001 0.001 0.001; visual mesh filename=../../meshes/shoulder_right_v1_1.stl scale=0.001 0.001 0.001
- link spine_default_1: geometry collision mesh filename=../../meshes/spine_default_1.stl scale=0.001 0.001 0.001; visual mesh filename=../../meshes/spine_default_1.stl scale=0.001 0.001 0.001
- link upper_arm_double_right_v1_1: geometry collision mesh filename=../../meshes/upper_arm_double_right_v1_1.stl scale=0.001 0.001 0.001; visual mesh filename=../../meshes/upper_arm_double_right_v1_1.stl scale=0.001 0.001 0.001
- link upper_arm_double_right_v1__1__1: geometry collision mesh filename=../../meshes/upper_arm_double_right_v1__1__1.stl scale=0.001 0.001 0.001; visual mesh filename=../../meshes/upper_arm_double_right_v1__1__1.stl scale=0.001 0.001 0.001

Commit message: edit urdf

File: urdf/Cogni-robot.urdf (robot description, URDF)
Before this commit: robot Cogni-robot, 36 links, 35 joints
Links:
- link Prehenseur_fifty_fifty_Main_right_v1_1: geometry collision mesh filename=meshes/Prehenseur_fifty_fifty_Main_right_v1_1.stl scale=0.001 0.001 0.001; visual mesh filename=meshes/Prehenseur_fifty_fifty_Main_right_v1_1.stl scale=0.001 0.001 0.001
- link Prehenseur_fifty_fifty_Main_right_v1__1__1: geometry collision mesh filename=meshes/Prehenseur_fifty_fifty_Main_right_v1__1__1.stl scale=0.001 0.001 0.001; visual mesh filename=meshes/Prehenseur_fifty_fifty_Main_right_v1__1__1.stl scale=0.001 0.001 0.001
- link Prehenseur_fifty_fifty_Pousse_right_v1_1: geometry collision mesh filename=meshes/Prehenseur_fifty_fifty_Pousse_right_v1_1.stl scale=0.001 0.001 0.001; visual mesh filename=meshes/Prehenseur_fifty_fifty_Pousse_right_v1_1.stl scale=0.001 0.001 0.001
- link Prehenseur_fifty_fifty_Pousse_right_v1__1__1: geometry collision mesh filename=meshes/Prehenseur_fifty_fifty_Pousse_right_v1__1__1.stl scale=0.001 0.001 0.001; visual mesh filename=meshes/Prehenseur_fifty_fifty_Pousse_right_v1__1__1.stl scale=0.001 0.001 0.001
- link arm_connector_Feetech_v1_1: geometry collision mesh filename=meshes/arm_connector_Feetech_v1_1.stl scale=0.001 0.001 0.001; visual mesh filename=meshes/arm_connector_Feetech_v1_1.stl scale=0.001 0.001 0.001
- link arm_connector_Feetech_v1__1__1: geometry collision mesh filename=meshes/arm_connector_Feetech_v1__1__1.stl scale=0.001 0.001 0.001; visual mesh filename=meshes/arm_connector_Feetech_v1__1__1.stl scale=0.001 0.001 0.001
- link avant_bras_left_1: geometry collision mesh filename=meshes/avant_bras_left_1.stl scale=0.001 0.001 0.001; visual mesh filename=meshes/avant_bras_left_1.stl scale=0.001 0.001 0.001
- link avant_bras_right_v1_1: geometry collision mesh filename=meshes/avant_bras_right_v1_1.stl scale=0.001 0.001 0.001; visual mesh filename=meshes/avant_bras_right_v1_1.stl scale=0.001 0.001 0.001
- link base_link: geometry collision mesh filename=meshes/base_link.stl scale=0.001 0.001 0.001; visual mesh filename=meshes/base_link.stl scale=0.001 0.001 0.001
- link chest_1: geometry collision mesh filename=meshes/chest_1.stl scale=0.001 0.001 0.001; visual mesh filename=meshes/chest_1.stl scale=0.001 0.001 0.001
- link double_rotation_link_double_feetech_v1_1: geometry collision mesh filename=meshes/double_rotation_link_double_feetech_v1_1.stl scale=0.001 0.001 0.001; visual mesh filename=meshes/double_rotation_link_double_feetech_v1_1.stl scale=0.001 0.001 0.001
- link double_rotation_link_double_feetech_v1__1__1: geometry collision mesh filename=meshes/double_rotation_link_double_feetech_v1__1__1.stl scale=0.001 0.001 0.001; visual mesh filename=meshes/double_rotation_link_double_feetech_v1__1__1.stl scale=0.001 0.001 0.001
- link head_back_v2_1: geometry collision mesh filename=meshes/head_back_v2_1.stl scale=0.001 0.001 0.001; visual mesh filename=meshes/head_back_v2_1.stl scale=0.001 0.001 0.001
- link head_face_v1_1: geometry collision mesh filename=meshes/head_face_v1_1.stl scale=0.001 0.001 0.001; visual mesh filename=meshes/head_face_v1_1.stl scale=0.001 0.001 0.001
- link neck_v2_1: geometry collision mesh filename=meshes/neck_v2_1.stl scale=0.001 0.001 0.001; visual mesh filename=meshes/neck_v2_1.stl scale=0.001 0.001 0.001
- link screen_v1_1: geometry collision mesh filename=meshes/screen_v1_1.stl scale=0.001 0.001 0.001; visual mesh filename=meshes/screen_v1_1.stl scale=0.001 0.001 0.001
- link servo-sts3215-2_1: geometry collision mesh filename=meshes/servo-sts3215-2_1.stl scale=0.001 0.001 0.001; visual mesh filename=meshes/servo-sts3215-2_1.stl scale=0.001 0.001 0.001
- link servo_sts3215-2_1: geometry collision mesh filename=meshes/servo_sts3215-2_1.stl scale=0.001 0.001 0.001; visual mesh filename=meshes/servo_sts3215-2_1.stl scale=0.001 0.001 0.001
- link servo_sts3215_v1_1: geometry collision mesh filename=meshes/servo_sts3215_v1_1.stl scale=0.001 0.001 0.001; visual mesh filename=meshes/servo_sts3215_v1_1.stl scale=0.001 0.001 0.001
- link servo_sts3215_v1__10__1: geometry collision mesh filename=meshes/servo_sts3215_v1__10__1.stl scale=0.001 0.001 0.001; visual mesh filename=meshes/servo_sts3215_v1__10__1.stl scale=0.001 0.001 0.001
- link servo_sts3215_v1__11__1: geometry collision mesh filename=meshes/servo_sts3215_v1__11__1.stl scale=0.001 0.001 0.001; visual mesh filename=meshes/servo_sts3215_v1__11__1.stl scale=0.001 0.001 0.001
- link servo_sts3215_v1__12__1: geometry collision mesh filename=meshes/servo_sts3215_v1__12__1.stl scale=0.001 0.001 0.001; visual mesh filename=meshes/servo_sts3215_v1__12__1.stl scale=0.001 0.001 0.001
- link servo_sts3215_v1__1__1: geometry collision mesh filename=meshes/servo_sts3215_v1__1__1.stl scale=0.001 0.001 0.001; visual mesh filename=meshes/servo_sts3215_v1__1__1.stl scale=0.001 0.001 0.001
- link servo_sts3215_v1__2__1: geometry collision mesh filename=meshes/servo_sts3215_v1__2__1.stl scale=0.001 0.001 0.001; visual mesh filename=meshes/servo_sts3215_v1__2__1.stl scale=0.001 0.001 0.001
- link servo_sts3215_v1__3__1: geometry collision mesh filename=meshes/servo_sts3215_v1__3__1.stl scale=0.001 0.001 0.001; visual mesh filename=meshes/servo_sts3215_v1__3__1.stl scale=0.001 0.001 0.001
- link servo_sts3215_v1__4__1: geometry collision mesh filename=meshes/servo_sts3215_v1__4__1.stl scale=0.001 0.001 0.001; visual mesh filename=meshes/servo_sts3215_v1__4__1.stl scale=0.001 0.001 0.001
- link servo_sts3215_v1__5__1: geometry collision mesh filename=meshes/servo_sts3215_v1__5__1.stl scale=0.001 0.001 0.001; visual mesh filename=meshes/servo_sts3215_v1__5__1.stl scale=0.001 0.001 0.001
- link servo_sts3215_v1__6__1: geometry collision mesh filename=meshes/servo_sts3215_v1__6__1.stl scale=0.001 0.001 0.001; visual mesh filename=meshes/servo_sts3215_v1__6__1.stl scale=0.001 0.001 0.001
- link servo_sts3215_v1__7__1: geometry collision mesh filename=meshes/servo_sts3215_v1__7__1.stl scale=0.001 0.001 0.001; visual mesh filename=meshes/servo_sts3215_v1__7__1.stl scale=0.001 0.001 0.001
- link servo_sts3215_v1__8__1: geometry collision mesh filename=meshes/servo_sts3215_v1__8__1.stl scale=0.001 0.001 0.001; visual mesh filename=meshes/servo_sts3215_v1__8__1.stl scale=0.001 0.001 0.001
- link servo_sts3215_v1__9__1: geometry collision mesh filename=meshes/servo_sts3215_v1__9__1.stl scale=0.001 0.001 0.001; visual mesh filename=meshes/servo_sts3215_v1__9__1.stl scale=0.001 0.001 0.001
- link shoulder_left_v1_1: geometry collision mesh filename=meshes/shoulder_left_v1_1.stl scale=0.001 0.001 0.001; visual mesh filename=meshes/shoulder_left_v1_1.stl scale=0.001 0.001 0.001
- link shoulder_right_v1_1: geometry collision mesh filename=meshes/shoulder_right_v1_1.stl scale=0.001 0.001 0.001; visual mesh filename=meshes/shoulder_right_v1_1.stl scale=0.001 0.001 0.001
- link spine_default_1: geometry collision mesh filename=meshes/spine_default_1.stl scale=0.001 0.001 0.001; visual mesh filename=meshes/spine_default_1.stl scale=0.001 0.001 0.001
- link upper_arm_double_right_v1_1: geometry collision mesh filename=meshes/upper_arm_double_right_v1_1.stl scale=0.001 0.001 0.001; visual mesh filename=meshes/upper_arm_double_right_v1_1.stl scale=0.001 0.001 0.001
- link upper_arm_double_right_v1__1__1: geometry collision mesh filename=meshes/upper_arm_double_right_v1__1__1.stl scale=0.001 0.001 0.001; visual mesh filename=meshes/upper_arm_double_right_v1__1__1.stl scale=0.001 0.001 0.001
