Commit message: Add Xacro processing script and update materials.xacro formatting
- Introduced a new Python script `xacro.py` for processing Xacro files, including handling includes, macros, and properties.
- Enhanced XML pretty printing for better readability.
- Updated `materials.xacro` to ensure proper formatting and structure.

File: urdf/Cogni-robot.urdf (robot description, URDF)
Before this commit: robot Cogni-robot, 36 links, 35 joints
Links:
- link Prehenseur_fifty_fifty_Main_right_v1_1: geometry collision mesh filename=Prehenseur_fifty_fifty_Main_right_v1_1.stl scale=0.001 0.001 0.001; visual mesh filename=Prehenseur_fifty_fifty_Main_right_v1_1.stl scale=0.001 0.001 0.001
- link Prehenseur_fifty_fifty_Main_right_v1__1__1: geometry collision mesh filename=Prehenseur_fifty_fifty_Main_right_v1__1__1.stl scale=0.001 0.001 0.001; visual mesh filename=Prehenseur_fifty_fifty_Main_right_v1__1__1.stl scale=0.001 0.001 0.001
- link Prehenseur_fifty_fifty_Pousse_right_v1_1: geometry collision mesh filename=Prehenseur_fifty_fifty_Pousse_right_v1_1.stl scale=0.001 0.001 0.001; visual mesh filename=Prehenseur_fifty_fifty_Pousse_right_v1_1.stl scale=0.001 0.001 0.001
- link Prehenseur_fifty_fifty_Pousse_right_v1__1__1: geometry collision mesh filename=Prehenseur_fifty_fifty_Pousse_right_v1__1__1.stl scale=0.001 0.001 0.001; visual mesh filename=Prehenseur_fifty_fifty_Pousse_right_v1__1__1.stl scale=0.001 0.001 0.001
- link arm_connector_Feetech_v1_1: geometry collision mesh filename=arm_connector_Feetech_v1_1.stl scale=0.001 0.001 0.001; visual mesh filename=arm_connector_Feetech_v1_1.stl scale=0.001 0.001 0.001
- link arm_connector_Feetech_v1__1__1: geometry collision mesh filename=arm_connector_Feetech_v1__1__1.stl scale=0.001 0.001 0.001; visual mesh filename=arm_connector_Feetech_v1__1__1.stl scale=0.001 0.001 0.001
- link avant_bras_left_1: geometry collision mesh filename=avant_bras_left_1.stl scale=0.001 0.001 0.001; visual mesh filename=avant_bras_left_1.stl scale=0.001 0.001 0.001
- link avant_bras_right_v1_1: geometry collision mesh filename=avant_bras_right_v1_1.stl scale=0.001 0.001 0.001; visual mesh filename=avant_bras_right_v1_1.stl scale=0.001 0.001 0.001
- link base_link: geometry collision mesh filename=base_link.stl scale=0.001 0.001 0.001; visual mesh filename=base_link.stl scale=0.001 0.001 0.001
- link chest_1: geometry collision mesh filename=chest_1.stl scale=0.001 0.001 0.001; visual mesh filename=chest_1.stl scale=0.001 0.001 0.001
- link double_rotation_link_double_feetech_v1_1: geometry collision mesh filename=double_rotation_link_double_feetech_v1_1.stl scale=0.001 0.001 0.001; visual mesh filename=double_rotation_link_double_feetech_v1_1.stl scale=0.001 0.001 0.001
- link double_rotation_link_double_feetech_v1__1__1: geometry collision mesh filename=double_rotation_link_double_feetech_v1__1__1.stl scale=0.001 0.001 0.001; visual mesh filename=double_rotation_link_double_feetech_v1__1__1.stl scale=0.001 0.001 0.001
- link head_back_v2_1: geometry collision mesh filename=head_back_v2_1.stl scale=0.001 0.001 0.001; visual mesh filename=head_back_v2_1.stl scale=0.001 0.001 0.001
- link head_face_v1_1: geometry collision mesh filename=head_face_v1_1.stl scale=0.001 0.001 0.001; visual mesh filename=head_face_v1_1.stl scale=0.001 0.001 0.001
- link neck_v2_1: geometry collision mesh filename=neck_v2_1.stl scale=0.001 0.001 0.001; visual mesh filename=neck_v2_1.stl scale=0.001 0.001 0.001
- link screen_v1_1: geometry collision mesh filename=screen_v1_1.stl scale=0.001 0.001 0.001; visual mesh filename=screen_v1_1.stl scale=0.001 0.001 0.001
- link servo-sts3215-2_1: geometry collision mesh filename=servo-sts3215-2_1.stl scale=0.001 0.001 0.001; visual mesh filename=servo-sts3215-2_1.stl scale=0.001 0.001 0.001
- link servo_sts3215-2_1: geometry collision mesh filename=servo_sts3215-2_1.stl scale=0.001 0.001 0.001; visual mesh filename=servo_sts3215-2_1.stl scale=0.001 0.001 0.001
- link servo_sts3215_v1_1: geometry collision mesh filename=servo_sts3215_v1_1.stl scale=0.001 0.001 0.001; visual mesh filename=servo_sts3215_v1_1.stl scale=0.001 0.001 0.001
- link servo_sts3215_v1__10__1: geometry collision mesh filename=servo_sts3215_v1__10__1.stl scale=0.001 0.001 0.001; visual mesh filename=servo_sts3215_v1__10__1.stl scale=0.001 0.001 0.001
- link servo_sts3215_v1__11__1: geometry collision mesh filename=servo_sts3215_v1__11__1.stl scale=0.001 0.001 0.001; visual mesh filename=servo_sts3215_v1__11__1.stl scale=0.001 0.001 0.001
- link servo_sts3215_v1__12__1: geometry collision mesh filename=servo_sts3215_v1__12__1.stl scale=0.001 0.001 0.001; visual mesh filename=servo_sts3215_v1__12__1.stl scale=0.001 0.001 0.001
- link servo_sts3215_v1__1__1: geometry collision mesh filename=servo_sts3215_v1__1__1.stl scale=0.001 0.001 0.001; visual mesh filename=servo_sts3215_v1__1__1.stl scale=0.001 0.001 0.001
- link servo_sts3215_v1__2__1: geometry collision mesh filename=servo_sts3215_v1__2__1.stl scale=0.001 0.001 0.001; visual mesh filename=servo_sts3215_v1__2__1.stl scale=0.001 0.001 0.001
- link servo_sts3215_v1__3__1: geometry collision mesh filename=servo_sts3215_v1__3__1.stl scale=0.001 0.001 0.001; visual mesh filename=servo_sts3215_v1__3__1.stl scale=0.001 0.001 0.001
- link servo_sts3215_v1__4__1: geometry collision mesh filename=servo_sts3215_v1__4__1.stl scale=0.001 0.001 0.001; visual mesh filename=servo_sts3215_v1__4__1.stl scale=0.001 0.001 0.001
- link servo_sts3215_v1__5__1: geometry collision mesh filename=servo_sts3215_v1__5__1.stl scale=0.001 0.001 0.001; visual mesh filename=servo_sts3215_v1__5__1.stl scale=0.001 0.001 0.001
- link servo_sts3215_v1__6__1: geometry collision mesh filename=servo_sts3215_v1__6__1.stl scale=0.001 0.001 0.001; visual mesh filename=servo_sts3215_v1__6__1.stl scale=0.001 0.001 0.001
- link servo_sts3215_v1__7__1: geometry collision mesh filename=servo_sts3215_v1__7__1.stl scale=0.001 0.001 0.001; visual mesh filename=servo_sts3215_v1__7__1.stl scale=0.001 0.001 0.001
- link servo_sts3215_v1__8__1: geometry collision mesh filename=servo_sts3215_v1__8__1.stl scale=0.001 0.001 0.001; visual mesh filename=servo_sts3215_v1__8__1.stl scale=0.001 0.001 0.001
- link servo_sts3215_v1__9__1: geometry collision mesh filename=servo_sts3215_v1__9__1.stl scale=0.001 0.001 0.001; visual mesh filename=servo_sts3215_v1__9__1.stl scale=0.001 0.001 0.001
- link shoulder_left_v1_1: geometry collision mesh filename=shoulder_left_v1_1.stl scale=0.001 0.001 0.001; visual mesh filename=shoulder_left_v1_1.stl scale=0.001 0.001 0.001
- link shoulder_right_v1_1: geometry collision mesh filename=shoulder_right_v1_1.stl scale=0.001 0.001 0.001; visual mesh filename=shoulder_right_v1_1.stl scale=0.001 0.001 0.001
- link spine_default_1: geometry collision mesh filename=spine_default_1.stl scale=0.001 0.001 0.001; visual mesh filename=spine_default_1.stl scale=0.001 0.001 0.001
- link upper_arm_double_right_v1_1: geometry collision mesh filename=upper_arm_double_right_v1_1.stl scale=0.001 0.001 0.001; visual mesh filename=upper_arm_double_right_v1_1.stl scale=0.001 0.001 0.001
- link upper_arm_double_right_v1__1__1: geometry collision mesh filename=upper_arm_double_right_v1__1__1.stl scale=0.001 0.001 0.001; visual mesh filename=upper_arm_double_right_v1__1__1.stl scale=0.001 0.001 0.001
Joints:
- removed joint Rigide 10
- removed joint Rigide 13
- removed joint Rigide 14
- removed joint Rigide 17
- removed joint Rigide 19
- removed joint Rigide 20
- removed joint Rigide 22
- removed joint Rigide 23
- removed joint Rigide 27
- removed joint Rigide 29
- removed joint Rigide 30
- removed joint Rigide 32
- removed joint Rigide 33
- removed joint Rigide 35
- removed joint Rigide 36
- removed joint Rigide 4
- removed joint Rigide 5
- removed joint Rigide 6
- removed joint Rigide 8
- removed joint Rigide 9
- removed joint rotation 34
- removed joint rotation 37
- removed joint rotation_bas_du_corps
- removed joint rotation_biceps_left
- removed joint rotation_biceps_right
- removed joint rotation_coude_left
- removed joint rotation_coude_right
- removed joint rotation_pince_right
- removed joint rotation_shoulder_xy_left
- removed joint rotation_shoulder_xy_right
- removed joint rotation_shoulder_zy_left
- removed joint rotation_soulder_zy_right
- removed joint rotation_yx_neck
- removed joint rotation_yx_torso
- removed joint rotation_zx_neck
- added joint elbow_left: type revolute, parent servo_sts3215_v1__11__1, child avant_bras_left_1, origin xyz=0.037386 -0.008496 0.004551 rpy=0 0 0, axis 0.0 -0.0 -1.0, limit lower=0.0 upper=2.40 effort=100 velocity=100
- added joint elbow_right: type revolute, parent servo_sts3215_v1__7__1, child avant_bras_right_v1_1, origin xyz=-0.031085 0.014996 0.004551 rpy=0 0 0, axis -0.0 -0.0 -1.0, limit lower=-2.4 upper=0.0 effort=100 velocity=100
- added joint fixed_10: type fixed, parent chest_1, child servo_sts3215-2_1, origin xyz=-0.010281 -0.052439 0.047526 rpy=0 0 0
- added joint fixed_13: type fixed, parent servo-sts3215-2_1, child head_back_v2_1, origin xyz=0.220532 -0.028617 0.060095 rpy=0 0 0
- added joint fixed_14: type fixed, parent head_back_v2_1, child head_face_v1_1, origin xyz=-0.239834 0.038658 0.032147 rpy=0 0 0
- added joint fixed_17: type fixed, parent servo_sts3215_v1__5__1, child arm_connector_Feetech_v1_1, origin xyz=-0.159121 -0.148625 -0.075992 rpy=0 0 0
- added joint fixed_19: type fixed, parent servo_sts3215_v1__6__1, child upper_arm_double_right_v1_1, origin xyz=0.172225 -0.170472 -0.065156 rpy=0 0 0
- added joint fixed_20: type fixed, parent upper_arm_double_right_v1_1, child servo_sts3215_v1__7__1, origin xyz=-0.248126 0.145236 0.080352 rpy=0 0 0
- added joint fixed_22: type fixed, parent avant_bras_right_v1_1, child servo_sts3215_v1__8__1, origin xyz=-0.090049 -0.01094 0.00858 rpy=0 0 0
- added joint fixed_23: type fixed, parent servo_sts3215_v1__8__1, child Prehenseur_fifty_fifty_Pousse_right_v1_1, origin xyz=0.057247 -0.149807 -0.37237 rpy=0 0 0
- added joint fixed_27: type fixed, parent servo_sts3215_v1__9__1, child arm_connector_Feetech_v1__1__1, origin xyz=-0.131532 -0.148625 0.075992 rpy=0 0 0
- added joint fixed_29: type fixed, parent servo_sts3215_v1__10__1, child upper_arm_double_right_v1__1__1, origin xyz=-0.172025 0.142882 0.082157 rpy=0 0 0
- added joint fixed_30: type fixed, parent upper_arm_double_right_v1__1__1, child servo_sts3215_v1__11__1, origin xyz=0.241626 -0.145968 -0.066944 rpy=0 0 0
- added joint fixed_32: type fixed, parent avant_bras_left_1, child servo_sts3215_v1__12__1, origin xyz=0.073594 0.204126 -0.366567 rpy=0 0 0
- added joint fixed_33: type fixed, parent servo_sts3215_v1__12__1, child Prehenseur_fifty_fifty_Pousse_right_v1__1__1, origin xyz=0.104844 -0.364483 0.7141 rpy=0 0 0
- added joint fixed_35: type fixed, parent head_face_v1_1, child screen_v1_1, origin xyz=-0.002749 -0.312936 -0.210216 rpy=0 0 0
- added joint fixed_36: type fixed, parent servo_sts3215_v1_1, child spine_default_1, origin xyz=-0.014996 -0.002914 0.034531 rpy=0 0 0
- added joint fixed_4: type fixed, parent servo_sts3215_v1__1__1, child double_rotation_link_double_feetech_v1_1, origin xyz=-0.00455 0.014996 0.014086 rpy=0 0 0
- added joint fixed_5: type fixed, parent servo_sts3215_v1__1__1, child double_rotation_link_double_feetech_v1__1__1, origin xyz=-0.034531 0.014996 -0.002914 rpy=0 0 0
- added joint fixed_6: type fixed, parent double_rotation_link_double_feetech_v1_1, child servo_sts3215_v1__2__1, origin xyz=-0.0001 0.0069 -0.017 rpy=0 0 0
- added joint fixed_8: type fixed, parent chest_1, child servo_sts3215_v1__3__1, origin xyz=0.072458 -0.189067 -0.071966 rpy=0 0 0
- added joint fixed_9: type fixed, parent chest_1, child servo_sts3215_v1__4__1, origin xyz=-0.075142 -0.189067 -0.071966 rpy=0 0 0
- added joint gripper_left: type revolute, parent servo_sts3215_v1__12__1, child Prehenseur_fifty_fifty_Main_right_v1__1__1, origin xyz=0.031451 -0.219416 0.372233 rpy=0 0 0, axis 0.0 1.0 -0.0, limit lower=-1.570796 upper=0.401426 effort=100 velocity=100
- added joint gripper_right: type revolute, parent servo_sts3215_v1__8__1, child Prehenseur_fifty_fifty_Main_right_v1_1, origin xyz=-0.015004 -0.004551 -0.002914 rpy=0 0 0, axis 0.0 1.0 -0.0, limit lower=-0.401426 upper=1.745329 effort=100 velocity=100
- added joint neck_pitch: type revolute, parent neck_v2_1, child servo-sts3215-2_1, origin xyz=0.017831 0.000119 0.020034 rpy=0 0 0, axis 1.0 -0.0 -0.0, limit lower=-0.45 upper=0.40 effort=100 velocity=100
- added joint neck_yaw: type revolute, parent servo_sts3215-2_1, child neck_v2_1, origin xyz=0.01025 -0.0083 0.0346 rpy=0 0 0, axis -0.0 -0.0 -1.0, limit lower=-1.832596 upper=1.919862 effort=100 velocity=100
- added joint shoulder_pitch_left: type revolute, parent shoulder_left_v1_1, child servo_sts3215_v1__9__1, origin xyz=0.03009 -0.009968 -8e-06 rpy=0 0 0, axis -0.0 -1.0 0.0, limit lower=-1.80 upper=1.67 effort=100 velocity=100
- added joint shoulder_pitch_right: type revolute, parent shoulder_right_v1_1, child servo_sts3215_v1__5__1, origin xyz=-0.03009 -0.009968 -8e-06 rpy=0 0 0, axis 0.0 1.0 -0.0, limit lower=-1.80 upper=1.67 effort=100 velocity=100
- added joint shoulder_roll_left: type revolute, parent servo_sts3215_v1__3__1, child shoulder_left_v1_1, origin xyz=0.005346 0.127748 0.123486 rpy=0 0 0, axis -1.0 0.0 -0.0, limit lower=-0.96 upper=3.926991 effort=100 velocity=100
- added joint shoulder_roll_right: type revolute, parent servo_sts3215_v1__4__1, child shoulder_right_v1_1, origin xyz=-0.002755 0.127748 0.123494 rpy=0 0 0, axis 1.0 -0.0 -0.0, limit lower=-3.93 upper=0.959931 effort=100 velocity=100
- added joint shoulder_yaw_left: type revolute, parent arm_connector_Feetech_v1__1__1, child servo_sts3215_v1__10__1, origin xyz=0.175717 0.178097 -0.076092 rpy=0 0 0, axis -1.0 0.0 0.0, limit lower=-1.570796 upper=1.658063 effort=100 velocity=100
- added joint shoulder_yaw_right: type revolute, parent arm_connector_Feetech_v1_1, child servo_sts3215_v1__6__1, origin xyz=0.114935 0.178097 0.076091 rpy=0 0 0, axis 1.0 -0.0 0.0, limit lower=-1.745329 upper=1.745329 effort=100 velocity=100
- added joint spine_roll: type revolute, parent spine_default_1, child servo_sts3215_v1__1__1, origin xyz=0.0334 0.001747 0.038861 rpy=0 0 0, axis 1.0 0.0 0.0, limit lower=-0.436332 upper=0.959931 effort=100 velocity=100
- added joint torso_pitch: type revolute, parent servo_sts3215_v1__2__1, child chest_1, origin xyz=-0.015004 0.034532 0.002914 rpy=0 0 0, axis 0.0 -1.0 0.0, limit lower=-0.698132 upper=0.785398 effort=100 velocity=100
- added joint torso_yaw: type revolute, parent base_link, child servo_sts3215_v1_1, origin xyz=2e-06 -0.064517 0.050918 rpy=0 0 0, axis 0.0 -0.0 -1.0, limit lower=-1.95 upper=1.95 effort=100 velocity=100
