Commit message: Add Xacro processing script and update materials.xacro formatting
- Introduced a new Python script `xacro.py` for processing Xacro files, including handling includes, macros, and properties.
- Enhanced XML pretty printing for better readability.
- Updated `materials.xacro` to ensure proper formatting and structure.

File: urdf/Cogni-robot.xacro (robot description, xacro)
@@ -1,10 +1,7 @@
 <?xml version="1.0" ?>
 <robot name="Cogni-robot" xmlns:xacro="http://www.ros.org/wiki/xacro">
-<xacro:include filename="$(find Cogni-robot_description)/urdf/materials.xacro" />
-<xacro:include filename="$(find Cogni-robot_description)/urdf/Cogni-robot.trans" />
-<xacro:include filename="$(find Cogni-robot_description)/urdf/Cogni-robot.gazebo" />
 <link name="base_link">
   <inertial>
-    <origin xyz="-1.1219501603328655e-05 -0.05652645349282051 -0.007126953017833521" rpy="0 0 0"/>
+    <origin xyz="-1.1219501603328655e-05 -0.056526453492820504 -0.007126953017833521" rpy="0 0 0"/>
     <mass value="1.2458370682377469"/>
     <inertia ixx="0.002516" iyy="0.00237" izz="0.002929" ixy="-7.5e-05" iyz="0.000124" ixz="5e-06"/>
@@ -13,5 +10,5 @@
     <origin xyz="0 0 0" rpy="0 0 0"/>
     <geometry>
-      <mesh filename="file://$(find Cogni-robot_description)/meshes/base_link.stl" scale="0.001 0.001 0.001"/>
+      <mesh filename="../meshes/base_link.stl" scale="0.001 0.001 0.001"/>
     </geometry>
     <material name="silver"/>
@@ -20,5 +17,5 @@
     <origin xyz="0 0 0" rpy="0 0 0"/>
     <geometry>
-      <mesh filename="file://$(find Cogni-robot_description)/meshes/base_link.stl" scale="0.001 0.001 0.001"/>
+      <mesh filename="../meshes/base_link.stl" scale="0.001 0.001 0.001"/>
     </geometry>
   </collision>
@@ -33,5 +30,5 @@
     <origin xyz="-2e-06 0.064517 -0.050918" rpy="0 0 0"/>
     <geometry>
-      <mesh filename="file://$(find Cogni-robot_description)/meshes/servo_sts3215_v1_1.stl" scale="0.001 0.001 0.001"/>
+      <mesh filename="../meshes/servo_sts3215_v1_1.stl" scale="0.001 0.001 0.001"/>
     </geometry>
     <material name="silver"/>
@@ -40,5 +37,5 @@
     <origin xyz="-2e-06 0.064517 -0.050918" rpy="0 0 0"/>
     <geometry>
-      <mesh filename="file://$(find Cogni-robot_description)/meshes/servo_sts3215_v1_1.stl" scale="0.001 0.001 0.001"/>
+      <mesh filename="../meshes/servo_sts3215_v1_1.stl" scale="0.001 0.001 0.001"/>
     </geometry>
   </collision>
@@ -53,5 +50,5 @@
     <origin xyz="-0.013856 0.050688 -0.138396" rpy="0 0 0"/>
     <geometry>
-      <mesh filename="file://$(find Cogni-robot_description)/meshes/double_rotation_link_double_feetech_v1_1.stl" scale="0.001 0.001 0.001"/>
+      <mesh filename="../meshes/double_rotation_link_double_feetech_v1_1.stl" scale="0.001 0.001 0.001"/>
     </geometry>
     <material name="silver"/>
@@ -60,5 +57,5 @@
     <origin xyz="-0.013856 0.050688 -0.138396" rpy="0 0 0"/>
     <geometry>
-      <mesh filename="file://$(find Cogni-robot_description)/meshes/double_rotation_link_double_feetech_v1_1.stl" scale="0.001 0.001 0.001"/>
+      <mesh filename="../meshes/double_rotation_link_double_feetech_v1_1.stl" scale="0.001 0.001 0.001"/>
     </geometry>
   </collision>
@@ -73,5 +70,5 @@
     <origin xyz="0.016125 0.050688 -0.121396" rpy="0 0 0"/>
     <geometry>
-      <mesh filename="file://$(find Cogni-robot_description)/meshes/double_rotation_link_double_feetech_v1__1__1.stl" scale="0.001 0.001 0.001"/>
+      <mesh filename="../meshes/double_rotation_link_double_feetech_v1__1__1.stl" scale="0.001 0.001 0.001"/>
     </geometry>
     <material name="silver"/>
@@ -80,5 +77,5 @@
     <origin xyz="0.016125 0.050688 -0.121396" rpy="0 0 0"/>
     <geometry>
-      <mesh filename="file://$(find Cogni-robot_description)/meshes/double_rotation_link_double_feetech_v1__1__1.stl" scale="0.001 0.001 0.001"/>
+      <mesh filename="../meshes/double_rotation_link_double_feetech_v1__1__1.stl" scale="0.001 0.001 0.001"/>
     </geometry>
   </collision>
@@ -93,5 +90,5 @@
     <origin xyz="-0.013756 0.043788 -0.121396" rpy="0 0 0"/>
     <geometry>
-      <mesh filename="file://$(find Cogni-robot_description)/meshes/servo_sts3215_v1__2__1.stl" scale="0.001 0.001 0.001"/>
+      <mesh filename="../meshes/servo_sts3215_v1__2__1.stl" scale="0.001 0.001 0.001"/>
     </geometry>
     <material name="silver"/>
@@ -100,5 +97,5 @@
     <origin xyz="-0.013756 0.043788 -0.121396" rpy="0 0 0"/>
     <geometry>
-      <mesh filename="file://$(find Cogni-robot_description)/meshes/servo_sts3215_v1__2__1.stl" scale="0.001 0.001 0.001"/>
+      <mesh filename="../meshes/servo_sts3215_v1__2__1.stl" scale="0.001 0.001 0.001"/>
     </geometry>
   </collision>
@@ -106,12 +103,12 @@
 <link name="chest_1">
   <inertial>
-    <origin xyz="0.0017826415962840523 -0.03577287736870712 0.04770661560159359" rpy="0 0 0"/>
+    <origin xyz="0.00015427959004198446 -0.03577287736870712 0.04773966957719847" rpy="0 0 0"/>
     <mass value="0.5907354450700422"/>
-    <inertia ixx="0.000784" iyy="0.001095" izz="0.001455" ixy="-1e-06" iyz="-1.5e-05" ixz="2.3e-05"/>
+    <inertia ixx="0.000783" iyy="0.001095" izz="0.001456" ixy="-0.0" iyz="-1.5e-05" ixz="-0.0"/>
   </inertial>
   <visual>
     <origin xyz="0.001248 0.009256 -0.12431" rpy="0 0 0"/>
     <geometry>
-      <mesh filename="file://$(find Cogni-robot_description)/meshes/chest_1.stl" scale="0.001 0.001 0.001"/>
+      <mesh filename="../meshes/chest_1.stl" scale="0.001 0.001 0.001"/>
     </geometry>
     <material name="silver"/>
@@ -120,5 +117,5 @@
     <origin xyz="0.001248 0.009256 -0.12431" rpy="0 0 0"/>
     <geometry>
-      <mesh filename="file://$(find Cogni-robot_description)/meshes/chest_1.stl" scale="0.001 0.001 0.001"/>
+      <mesh filename="../meshes/chest_1.stl" scale="0.001 0.001 0.001"/>
     </geometry>
   </collision>
@@ -126,19 +123,19 @@
 <link name="servo_sts3215_v1__3__1">
   <inertial>
-    <origin xyz="-0.01077308895703491 0.13907074034428557 0.12394977494486209" rpy="0 0 0"/>
-    <mass value="0.34332301760825074"/>
-    <inertia ixx="9.2e-05" iyy="5.8e-05" izz="9.9e-05" ixy="1e-06" iyz="0.0" ixz="0.0"/>
-  </inertial>
-  <visual>
-    <origin xyz="-0.070938 0.195769 -0.049838" rpy="0 0 0"/>
-    <geometry>
-      <mesh filename="file://$(find Cogni-robot_description)/meshes/servo_sts3215_v1__3__1.stl" scale="0.001 0.001 0.001"/>
-    </geometry>
-    <material name="silver"/>
-  </visual>
-  <collision>
-    <origin xyz="-0.070938 0.195769 -0.049838" rpy="0 0 0"/>
-    <geometry>
-      <mesh filename="file://$(find Cogni-robot_description)/meshes/servo_sts3215_v1__3__1.stl" scale="0.001 0.001 0.001"/>
+    <origin xyz="-0.012768569454018337 0.14162474034428557 0.12350985679084983" rpy="0 0 0"/>
+    <mass value="0.34332301760825074"/>
+    <inertia ixx="9.2e-05" iyy="5.8e-05" izz="9.9e-05" ixy="1e-06" iyz="0.0" ixz="-0.0"/>
+  </inertial>
+  <visual>
+    <origin xyz="-0.07121 0.198323 -0.052344" rpy="0 0 0"/>
+    <geometry>
+      <mesh filename="../meshes/servo_sts3215_v1__3__1.stl" scale="0.001 0.001 0.001"/>
+    </geometry>
+    <material name="silver"/>
+  </visual>
+  <collision>
+    <origin xyz="-0.07121 0.198323 -0.052344" rpy="0 0 0"/>
+    <geometry>
+      <mesh filename="../meshes/servo_sts3215_v1__3__1.stl" scale="0.001 0.001 0.001"/>
     </geometry>
   </collision>
@@ -146,19 +143,19 @@
 <link name="servo_sts3215_v1__4__1">
   <inertial>
-    <origin xyz="0.01725059524034419 0.14410574034429674 0.12295290509015946" rpy="0 0 0"/>
-    <mass value="0.34332301760825074"/>
-    <inertia ixx="9.2e-05" iyy="5.8e-05" izz="9.9e-05" ixy="-1e-06" iyz="-0.0" ixz="0.0"/>
-  </inertial>
-  <visual>
-    <origin xyz="0.07649 0.200804 -0.05487" rpy="0 0 0"/>
-    <geometry>
-      <mesh filename="file://$(find Cogni-robot_description)/meshes/servo_sts3215_v1__4__1.stl" scale="0.001 0.001 0.001"/>
-    </geometry>
-    <material name="silver"/>
-  </visual>
-  <collision>
-    <origin xyz="0.07649 0.200804 -0.05487" rpy="0 0 0"/>
-    <geometry>
-      <mesh filename="file://$(find Cogni-robot_description)/meshes/servo_sts3215_v1__4__1.stl" scale="0.001 0.001 0.001"/>
+    <origin xyz="0.01535895970710844 0.14162474034429673 0.12346961705796619" rpy="0 0 0"/>
+    <mass value="0.34332301760825074"/>
+    <inertia ixx="9.2e-05" iyy="5.8e-05" izz="9.9e-05" ixy="-1e-06" iyz="-0.0" ixz="-0.0"/>
+  </inertial>
+  <visual>
+    <origin xyz="0.07639 0.198323 -0.052344" rpy="0 0 0"/>
+    <geometry>
+      <mesh filename="../meshes/servo_sts3215_v1__4__1.stl" scale="0.001 0.001 0.001"/>
+    </geometry>
+    <material name="silver"/>
+  </visual>
+  <collision>
+    <origin xyz="0.07639 0.198323 -0.052344" rpy="0 0 0"/>
+    <geometry>
+      <mesh filename="../meshes/servo_sts3215_v1__4__1.stl" scale="0.001 0.001 0.001"/>
     </geometry>
   </collision>
@@ -166,19 +163,19 @@
 <link name="servo_sts3215-2_1">
   <inertial>
-    <origin xyz="0.01080377387017686 0.004721873144410228 0.016041191549275413" rpy="0 0 0"/>
+    <origin xyz="0.010250157404470425 0.004721873144410249 0.016400350717485745" rpy="0 0 0"/>
     <mass value="0.2747881442151801"/>
-    <inertia ixx="7.1e-05" iyy="3.8e-05" izz="6e-05" ixy="0.0" iyz="1e-06" ixz="-0.0"/>
-  </inertial>
-  <visual>
-    <origin xyz="0.009902 0.061695 -0.172159" rpy="0 0 0"/>
-    <geometry>
-      <mesh filename="file://$(find Cogni-robot_description)/meshes/servo_sts3215-2_1.stl" scale="0.001 0.001 0.001"/>
-    </geometry>
-    <material name="silver"/>
-  </visual>
-  <collision>
-    <origin xyz="0.009902 0.061695 -0.172159" rpy="0 0 0"/>
-    <geometry>
-      <mesh filename="file://$(find Cogni-robot_description)/meshes/servo_sts3215-2_1.stl" scale="0.001 0.001 0.001"/>
+    <inertia ixx="7.1e-05" iyy="3.8e-05" izz="6e-05" ixy="-0.0" iyz="1e-06" ixz="0.0"/>
+  </inertial>
+  <visual>
+    <origin xyz="0.011529 0.061695 -0.171836" rpy="0 0 0"/>
+    <geometry>
+      <mesh filename="../meshes/servo_sts3215-2_1.stl" scale="0.001 0.001 0.001"/>
+    </geometry>
+    <material name="silver"/>
+  </visual>
+  <collision>
+    <origin xyz="0.011529 0.061695 -0.171836" rpy="0 0 0"/>
+    <geometry>
+      <mesh filename="../meshes/servo_sts3215-2_1.stl" scale="0.001 0.001 0.001"/>
     </geometry>
   </collision>
@@ -186,19 +183,19 @@
 <link name="neck_v2_1">
   <inertial>
-    <origin xyz="0.0011067108619048087 -7.796325199518894e-05 0.010446641628047398" rpy="0 0 0"/>
+    <origin xyz="0.0007485223224610761 -9.349216530497861e-05 0.01047807820130392" rpy="0 0 0"/>
     <mass value="0.056145921126082916"/>
-    <inertia ixx="7e-06" iyy="2.5e-05" izz="2.2e-05" ixy="-0.0" iyz="0.0" ixz="0.0"/>
-  </inertial>
-  <visual>
-    <origin xyz="-0.001523 0.069995 -0.206389" rpy="0 0 0"/>
-    <geometry>
-      <mesh filename="file://$(find Cogni-robot_description)/meshes/neck_v2_1.stl" scale="0.001 0.001 0.001"/>
-    </geometry>
-    <material name="silver"/>
-  </visual>
-  <collision>
-    <origin xyz="-0.001523 0.069995 -0.206389" rpy="0 0 0"/>
-    <geometry>
-      <mesh filename="file://$(find Cogni-robot_description)/meshes/neck_v2_1.stl" scale="0.001 0.001 0.001"/>
+    <inertia ixx="7e-06" iyy="2.5e-05" izz="2.2e-05" ixy="-0.0" iyz="0.0" ixz="-0.0"/>
+  </inertial>
+  <visual>
+    <origin xyz="0.001279 0.069995 -0.206436" rpy="0 0 0"/>
+    <geometry>
+      <mesh filename="../meshes/neck_v2_1.stl" scale="0.001 0.001 0.001"/>
+    </geometry>
+    <material name="silver"/>
+  </visual>
+  <collision>
+    <origin xyz="0.001279 0.069995 -0.206436" rpy="0 0 0"/>
+    <geometry>
+      <mesh filename="../meshes/neck_v2_1.stl" scale="0.001 0.001 0.001"/>
     </geometry>
   </collision>
@@ -206,19 +203,19 @@
 <link name="servo-sts3215-2_1">
   <inertial>
-    <origin xyz="-0.018247862675479898 0.011480432576153853 0.006002529329745765" rpy="0 0 0"/>
+    <origin xyz="-0.018200236746651933 0.01185966221025403 0.005376001252874213" rpy="0 0 0"/>
     <mass value="0.2747881442151801"/>
     <inertia ixx="6e-05" iyy="4.3e-05" izz="6.5e-05" ixy="1e-06" iyz="-1.2e-05" ixz="1e-06"/>
   </inertial>
   <visual>
-    <origin xyz="-0.02002 0.069507 -0.225803" rpy="0 0 0"/>
-    <geometry>
-      <mesh filename="file://$(find Cogni-robot_description)/meshes/servo-sts3215-2_1.stl" scale="0.001 0.001 0.001"/>
-    </geometry>
-    <material name="silver"/>
-  </visual>
-  <collision>
-    <origin xyz="-0.02002 0.069507 -0.225803" rpy="0 0 0"/>
-    <geometry>
-      <mesh filename="file://$(find Cogni-robot_description)/meshes/servo-sts3215-2_1.stl" scale="0.001 0.001 0.001"/>
+    <origin xyz="-0.016552 0.069876 -0.22647" rpy="0 0 0"/>
+    <geometry>
+      <mesh filename="../meshes/servo-sts3215-2_1.stl" scale="0.001 0.001 0.001"/>
+    </geometry>
+    <material name="silver"/>
+  </visual>
+  <collision>
+    <origin xyz="-0.016552 0.069876 -0.22647" rpy="0 0 0"/>
+    <geometry>
+      <mesh filename="../meshes/servo-sts3215-2_1.stl" scale="0.001 0.001 0.001"/>
     </geometry>
   </collision>
@@ -226,19 +223,19 @@
 <link name="head_back_v2_1">
   <inertial>
-    <origin xyz="-0.2412539502615543 0.06385288729086241 -0.00924470605963662" rpy="0 0 0"/>
+    <origin xyz="-0.2399997142999622 0.06546375235283343 -0.019336533745128448" rpy="0 0 0"/>
     <mass value="0.5424516303112991"/>
-    <inertia ixx="0.000841" iyy="0.001374" izz="0.001028" ixy="-1.8e-05" iyz="-8.9e-05" ixz="4e-06"/>
-  </inertial>
-  <visual>
-    <origin xyz="-0.242449 0.096924 -0.276473" rpy="0 0 0"/>
-    <geometry>
-      <mesh filename="file://$(find Cogni-robot_description)/meshes/head_back_v2_1.stl" scale="0.001 0.001 0.001"/>
-    </geometry>
-    <material name="silver"/>
-  </visual>
-  <collision>
-    <origin xyz="-0.242449 0.096924 -0.276473" rpy="0 0 0"/>
-    <geometry>
-      <mesh filename="file://$(find Cogni-robot_description)/meshes/head_back_v2_1.stl" scale="0.001 0.001 0.001"/>
+    <inertia ixx="0.00084" iyy="0.001375" izz="0.001028" ixy="-4e-06" iyz="-9e-05" ixz="-5e-06"/>
+  </inertial>
+  <visual>
+    <origin xyz="-0.237084 0.098493 -0.286565" rpy="0 0 0"/>
+    <geometry>
+      <mesh filename="../meshes/head_back_v2_1.stl" scale="0.001 0.001 0.001"/>
+    </geometry>
+    <material name="silver"/>
+  </visual>
+  <collision>
+    <origin xyz="-0.237084 0.098493 -0.286565" rpy="0 0 0"/>
+    <geometry>
+      <mesh filename="../meshes/head_back_v2_1.stl" scale="0.001 0.001 0.001"/>
     </geometry>
   </collision>
@@ -246,19 +243,19 @@
 <link name="head_face_v1_1">
   <inertial>
-    <origin xyz="-0.0013476295627852775 -0.028179818730380383 -0.05660827912780514" rpy="0 0 0"/>
+    <origin xyz="-4.459929631812562e-08 -0.028186198727073175 -0.056621570075358396" rpy="0 0 0"/>
     <mass value="0.3123301638656947"/>
-    <inertia ixx="0.000532" iyy="0.001043" izz="0.00067" ixy="-1.4e-05" iyz="-9.1e-05" ixz="7e-06"/>
-  </inertial>
-  <visual>
-    <origin xyz="-0.003672 0.059868 -0.318657" rpy="0 0 0"/>
-    <geometry>
-      <mesh filename="file://$(find Cogni-robot_description)/meshes/head_face_v1_1.stl" scale="0.001 0.001 0.001"/>
-    </geometry>
-    <material name="silver"/>
-  </visual>
-  <collision>
-    <origin xyz="-0.003672 0.059868 -0.318657" rpy="0 0 0"/>
-    <geometry>
-      <mesh filename="file://$(find Cogni-robot_description)/meshes/head_face_v1_1.stl" scale="0.001 0.001 0.001"/>
+    <inertia ixx="0.000531" iyy="0.001043" izz="0.000671" ixy="-0.0" iyz="-9.1e-05" ixz="-0.0"/>
+  </inertial>
+  <visual>
+    <origin xyz="0.00275 0.059835 -0.318712" rpy="0 0 0"/>
+    <geometry>
+      <mesh filename="../meshes/head_face_v1_1.stl" scale="0.001 0.001 0.001"/>
+    </geometry>
+    <material name="silver"/>
+  </visual>
+  <collision>
+    <origin xyz="0.00275 0.059835 -0.318712" rpy="0 0 0"/>
+    <geometry>
+      <mesh filename="../meshes/head_face_v1_1.stl" scale="0.001 0.001 0.001"/>
     </geometry>
   </collision>
@@ -266,19 +263,19 @@
 <link name="shoulder_right_v1_1">
   <inertial>
-    <origin xyz="-0.013010640630053832 0.007820696038384783 0.001876770495154445" rpy="0 0 0"/>
+    <origin xyz="-0.01306709110545963 0.007820696038384783 0.0014317075357701825" rpy="0 0 0"/>
     <mass value="0.0899660706083263"/>
-    <inertia ixx="3.4e-05" iyy="2.1e-05" izz="3.9e-05" ixy="0.0" iyz="-0.0" ixz="-0.0"/>
-  </inertial>
-  <visual>
-    <origin xyz="0.077342 0.070575 -0.178465" rpy="0 0 0"/>
-    <geometry>
-      <mesh filename="file://$(find Cogni-robot_description)/meshes/shoulder_right_v1_1.stl" scale="0.001 0.001 0.001"/>
-    </geometry>
-    <material name="silver"/>
-  </visual>
-  <collision>
-    <origin xyz="0.077342 0.070575 -0.178465" rpy="0 0 0"/>
-    <geometry>
-      <mesh filename="file://$(find Cogni-robot_description)/meshes/shoulder_right_v1_1.stl" scale="0.001 0.001 0.001"/>
+    <inertia ixx="3.4e-05" iyy="2.1e-05" izz="3.9e-05" ixy="0.0" iyz="-0.0" ixz="-1e-06"/>
+  </inertial>
+  <visual>
+    <origin xyz="0.079145 0.070575 -0.175838" rpy="0 0 0"/>
+    <geometry>
+      <mesh filename="../meshes/shoulder_right_v1_1.stl" scale="0.001 0.001 0.001"/>
+    </geometry>
+    <material name="silver"/>
+  </visual>
+  <collision>
+    <origin xyz="0.079145 0.070575 -0.175838" rpy="0 0 0"/>
+    <geometry>
+      <mesh filename="../meshes/shoulder_right_v1_1.stl" scale="0.001 0.001 0.001"/>
     </geometry>
   </collision>
@@ -286,19 +283,19 @@
 <link name="servo_sts3215_v1__5__1">
   <inertial>
-    <origin xyz="-0.0004493364601803884 0.01811472819165904 -0.013869550088784072" rpy="0 0 0"/>
-    <mass value="0.34332301760825074"/>
-    <inertia ixx="9.8e-05" iyy="9.2e-05" izz="5.8e-05" ixy="0.0" iyz="1e-06" ixz="-1e-06"/>
-  </inertial>
-  <visual>
-    <origin xyz="0.107415 0.080543 -0.179483" rpy="0 0 0"/>
-    <geometry>
-      <mesh filename="file://$(find Cogni-robot_description)/meshes/servo_sts3215_v1__5__1.stl" scale="0.001 0.001 0.001"/>
-    </geometry>
-    <material name="silver"/>
-  </visual>
-  <collision>
-    <origin xyz="0.107415 0.080543 -0.179483" rpy="0 0 0"/>
-    <geometry>
-      <mesh filename="file://$(find Cogni-robot_description)/meshes/servo_sts3215_v1__5__1.stl" scale="0.001 0.001 0.001"/>
+    <origin xyz="-0.013877451272128485 0.01811472819166042 -2.4511628808843167e-05" rpy="0 0 0"/>
+    <mass value="0.34332301760825074"/>
+    <inertia ixx="5.8e-05" iyy="9.2e-05" izz="9.9e-05" ixy="1e-06" iyz="-0.0" ixz="0.0"/>
+  </inertial>
+  <visual>
+    <origin xyz="0.109235 0.080543 -0.17583" rpy="0 0 0"/>
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
Commit message: Rename body and joint elements in URDF and XML for consistency and clarity

File: urdf/Cogni-robot.urdf (robot description, URDF)
Before this commit: robot Cogni-robot, 36 links, 35 joints
Links:
- removed link head_face_v1_1
- removed link servo-sts3215-2_1
- added link head_face, mass 0.3123301638656947; collision mesh filename=head_face_v1_1.stl scale=0.001 0.001 0.001; visual mesh filename=head_face_v1_1.stl scale=0.001 0.001 0.001
- added link tete, mass 0.2747881442151801; collision mesh filename=servo-sts3215-2_1.stl scale=0.001 0.001 0.001; visual mesh filename=servo-sts3215-2_1.stl scale=0.001 0.001 0.001
Joints:
- joint fixed_13: parent servo-sts3215-2_1 -> tete
- joint fixed_14: child head_face_v1_1 -> head_face
- joint fixed_35: parent head_face_v1_1 -> head_face
- joint neck_pitch: child servo-sts3215-2_1 -> tete
